Commit message: add camera

File: model/robot.xacro (robot description, xacro)
@@ -1,11 +1,9 @@
 <?xml version="1.0"?>
 <robot name="differential_drive_robot" xmlns:xacro="http://www.ros.org/wiki/xacro">
-    <!-- Robot Parameters -->
     <xacro:property name="PI" value="3.14159265"/>
-    <xacro:property name="body_length" value="0.5"/>
-    <xacro:property name="body_width" value="0.3"/>
+    <xacro:property name="body_length" value="1.0"/>
+    <xacro:property name="body_width" value="1.0"/>
     <xacro:property name="body_height" value="0.1"/>
-    <xacro:property name="body_density" value="7850.0"/> <!-- Steel -->
-    <xacro:property name="body_mass" value="${body_density * body_length * body_height * body_width}"/>
+    <xacro:property name="body_density" value="7850.0"/> <xacro:property name="body_mass" value="${body_density * body_length * body_height * body_width}"/>
     <xacro:property name="body_inertia_x" value="${1.0/12.0 * body_mass * (body_height*body_height + body_width*body_width)}"/>
     <xacro:property name="body_inertia_y" value="${1.0/12.0 * body_mass * (body_length*body_length + body_height*body_height)}"/>
@@ -15,6 +13,5 @@
     <xacro:property name="wheel_separation" value="${body_width + wheel_width}"/>
     <xacro:property name="wheel_offset" value="${body_length/2 - wheel_radius}"/>
-    <xacro:property name="wheel_density" value="900"/> <!-- Ruber -->
-    <xacro:property name="wheel_mass" value="${wheel_density * PI * wheel_radius * wheel_radius * wheel_width}"/>
+    <xacro:property name="wheel_density" value="900"/> <xacro:property name="wheel_mass" value="${wheel_density * PI * wheel_radius * wheel_radius * wheel_width}"/>
     <xacro:property name="wheel_inertia_x" value="${1.0/12.0 * wheel_mass * (3*wheel_radius*wheel_radius + wheel_width*wheel_width)}"/>
     <xacro:property name="wheel_inertia_y" value="${1.0/12.0 * wheel_mass * (3*wheel_radius*wheel_radius + wheel_width*wheel_width)}"/>
@@ -27,8 +24,5 @@
     <xacro:property name="caster_inertia_y" value="${2.0/5.0 * caster_mass * caster_radius * caster_radius}"/>
     <xacro:property name="caster_inertia_z" value="${2.0/5.0 * caster_mass * caster_radius * caster_radius}"/>
-    <!-- Control Parameters -->
     <xacro:property name="max_linear_acceleration" value="10"/>
-    <!-- Links -->
-    <!-- Body Link -->
     <link name="body_link">
         <visual>
@@ -53,5 +47,4 @@
         </inertial>
     </link>
-    <!-- Left Wheel -->
     <link name="left_wheel_link">
         <visual>
@@ -76,5 +69,4 @@
         </inertial>
     </link>
-    <!-- Right Wheel -->
     <link name="right_wheel_link">
         <visual>
@@ -99,5 +91,4 @@
         </inertial>
     </link>
-    <!-- Caster Wheel -->
     <link name="caster_link">
         <visual>
@@ -122,6 +113,4 @@
         </inertial>
     </link>
-    <!-- Joints -->
-    <!-- Left Wheel Joint -->
     <joint name="left_wheel_joint" type="continuous">
         <origin xyz="-${wheel_offset} ${wheel_separation/2} -${wheel_radius/2}" rpy="0 0 0"/>
@@ -132,5 +121,4 @@
         <dynamics damping="0.1" friction="0.1"/>
     </joint>
-    <!-- Right Wheel Joint -->
     <joint name="right_wheel_joint" type="continuous">
         <origin xyz="-${wheel_offset} ${-wheel_separation/2} -${wheel_radius/2}" rpy="0 0 0"/>
@@ -141,5 +129,4 @@
         <dynamics damping="0.1" friction="0.1"/>
     </joint>
-    <!-- Caster Wheel Joint (fixed) -->
     <joint name="caster_joint" type="fixed">
         <origin xyz="${caster_offset} 0 -${caster_radius/2}" rpy="0 0 0"/>
@@ -147,5 +134,4 @@
         <child link="caster_link"/>
     </joint>
-    <!-- Gazebo Parameters -->
     <gazebo reference="body_link">
         <mu1>1.0</mu1>
@@ -164,5 +150,4 @@
         <mu2>0.000001</mu2>
     </gazebo>
-    <!-- Gazebo Plugins -->
     <gazebo>
         <plugin filename="gz-sim-diff-drive-system" name="gz::sim::systems::DiffDrive">
@@ -182,3 +167,4 @@
         </plugin>
     </gazebo>
+    <xacro:include filename="camera.xacro" />
 </robot>
